Commit message: updated spawn error

File: car_and_trailer/urdf/car_and_trailer.urdf.xacro (robot description, xacro)
@@ -1,7 +1,8 @@
-<?xml version="1.0" ?>
+<?xml version="1.0"?>
 <!-- This URDF was automatically created by SolidWorks to URDF Exporter! Originally created by Stephen Brawner (brawner@gmail.com)
      Commit Version: 1.6.0-4-g7f85cfe  Build Version: 1.6.7995.38578
      For more information, please see http://wiki.ros.org/sw_urdf_exporter -->
-<robot name="car_and_trailer" xmlns:xacro="http://ros.org/wiki/xacro">
+<robot
+  name="car_and_trailer" xmlns:xacro="http://ros.org/wiki/xacro">
   <link
     name="base_link">
@@ -11,9 +12,9 @@
         rpy="0 0 0" />
       <mass
-        value="10" />
-      <inertia
-        ixx="4.7150458258324"
-        ixy="-9.46382342562312E-17"
-        ixz="-1.15879432428749E-16"
+        value="45.8674211610964" />
+      <inertia
+        ixx="4.71504582583239"
+        ixy="-7.73092194649668E-17"
+        ixz="-1.15927084096081E-16"
         iyy="1.08472485190803"
         iyz="-0.316618072863205"
@@ -53,10 +54,10 @@
         value="0.205068851277686" />
       <inertia
-        ixx="0.000542814148788583"
-        ixy="8.06604141671555E-20"
-        ixz="-7.80565059903452E-05"
+        ixx="0.000542814148788568"
+        ixy="8.49018783728658E-19"
+        ixz="-7.80565059903451E-05"
         iyy="0.000546349438812291"
-        iyz="4.3660867095781E-19"
-        izz="9.40760107910967E-05" />
+        iyz="1.09592188639126E-18"
+        izz="9.40760107910819E-05" />
     </inertial>
     <visual>
@@ -86,8 +87,8 @@
   <joint
     name="Left_Steer"
-    type="continuous">
+    type="fixed">
     <origin
       xyz="0.508 2.0066 0"
-      rpy="3.1416 0 0" />
+      rpy="3.14159265358979 0 0" />
     <parent
       link="base_link" />
@@ -95,5 +96,5 @@
       link="Steer_Left" />
     <axis
-      xyz="0 0 1" />
+      xyz="0 0 0" />
   </joint>
   <link
@@ -142,5 +143,5 @@
     <origin
       xyz="-0.4826 1.0033 0.1651"
-      rpy="-1.5708 0 -1.5708" />
+      rpy="-1.5707963267949 0 -1.5707963267949" />
     <parent
       link="Steer_Left" />
@@ -160,8 +161,8 @@
       <inertia
         ixx="0.000542814148788574"
-        ixy="3.02286543581972E-20"
+        ixy="3.00990364412103E-20"
         ixz="-7.80565059903447E-05"
         iyy="0.00054634943881229"
-        iyz="3.76125579916017E-20"
+        iyz="3.72059530276015E-20"
         izz="9.4076010791088E-05" />
     </inertial>
@@ -192,8 +193,8 @@
   <joint
     name="Rigth_Steer"
-    type="continuous">
+    type="fixed">
     <origin
       xyz="0 0 0"
-      rpy="3.1416 0 3.1416" />
+      rpy="3.14159265358979 0 3.14159265358979" />
     <parent
       link="base_link" />
@@ -201,5 +202,5 @@
       link="Steer_Right" />
     <axis
-      xyz="0 0 1" />
+      xyz="0 0 0" />
   </joint>
   <link
@@ -208,4 +209,57 @@
       <origin
         xyz="0 0 0.0254"
+        rpy="0 0 0" />
+      <mass
+        value="1.62962959682594" />
+      <inertia
+        ixx="0.0046013275103996"
+        ixy="-7.56314231045415E-39"
+        ixz="-4.17161150360145E-36"
+        iyy="0.0046013275103996"
+        iyz="-8.30428564488929E-36"
+        izz="0.00850174046700706" />
+    </inertial>
+    <visual>
+      <origin
+        xyz="0 0 0"
+        rpy="0 0 0" />
+      <geometry>
+        <mesh
+          filename="package://car_and_trailer/meshes/Rigth_Front_Wheel.STL" />
+      </geometry>
+      <material
+        name="">
+        <color
+          rgba="0.792156862745098 0.819607843137255 0.933333333333333 1" />
+      </material>
+    </visual>
+    <collision>
+      <origin
+        xyz="0 0 0"
+        rpy="0 0 0" />
+      <geometry>
+        <mesh
+          filename="package://car_and_trailer/meshes/Rigth_Front_Wheel.STL" />
+      </geometry>
+    </collision>
+  </link>
+  <joint
+    name="Rigth_Front_Wheel_joint"
+    type="continuous">
+    <origin
+      xyz="-0.4826 1.0033 0.1651"
+      rpy="3.14159265358979 -1.5707963267949 0" />
+    <parent
+      link="Steer_Right" />
+    <child
+      link="Rigth_Front_Wheel" />
+    <axis
+      xyz="0 0 1" />
+  </joint>
+  <link
+    name="Right_Back_Wheel">
+    <inertial>
+      <origin
+        xyz="-6.93889390390723E-18 1.38777878078145E-16 0.0254"
         rpy="0 0 0" />
       <mass
@@ -225,57 +279,4 @@
       <geometry>
         <mesh
-          filename="package://car_and_trailer/meshes/Rigth_Front_Wheel.STL" />
-      </geometry>
-      <material
-        name="">
-        <color
-          rgba="0.792156862745098 0.819607843137255 0.933333333333333 1" />
-      </material>
-    </visual>
-    <collision>
-      <origin
-        xyz="0 0 0"
-        rpy="0 0 0" />
-      <geometry>
-        <mesh
-          filename="package://car_and_trailer/meshes/Rigth_Front_Wheel.STL" />
-      </geometry>
-    </collision>
-  </link>
-  <joint
-    name="Rigth_Front_Wheel_joint"
-    type="continuous">
-    <origin
-      xyz="-0.4826 1.0033 0.1651"
-      rpy="3.1416 -1.5708 0" />
-    <parent
-      link="Steer_Right" />
-    <child
-      link="Rigth_Front_Wheel" />
-    <axis
-      xyz="0 0 1" />
-  </joint>
-  <link
-    name="Right_Back_Wheel">
-    <inertial>
-      <origin
-        xyz="-6.93889390390723E-18 1.38777878078145E-16 0.0254"
-        rpy="0 0 0" />
-      <mass
-        value="1.62962959682594" />
-      <inertia
-        ixx="0.0046013275103996"
-        ixy="-7.56314231045415E-39"
-        ixz="-4.17161150360145E-36"
-        iyy="0.0046013275103996"
-        iyz="-8.30428564488929E-36"
-        izz="0.00850174046700706" />
-    </inertial>
-    <visual>
-      <origin
-        xyz="0 0 0"
-        rpy="0 0 0" />
-      <geometry>
-        <mesh
           filename="package://car_and_trailer/meshes/Right_Back_Wheel.STL" />
       </geometry>
@@ -300,6 +301,6 @@
     type="continuous">
     <origin
-      xyz="0.4826 0.0381 -0.1651"
-      rpy="1.5708 0 1.5708" />
+      xyz="0.4826 0.0381000000000003 -0.1651"
+      rpy="1.5707963267949 0 1.5707963267949" />
     <parent
       link="base_link" />
@@ -353,6 +354,6 @@
     type="continuous">
     <origin
-      xyz="0 0.0381 -0.1651"
-      rpy="1.5708 0 1.5708" />
+      xyz="0 0.0381000000000003 -0.1651"
+      rpy="1.5707963267949 0 1.5707963267949" />
     <parent
       link="base_link" />
@@ -419,15 +420,15 @@
     <inertial>
       <origin
-        xyz="5.55111512312578E-17 -0.487159812610342 0.0270212640980216"
-        rpy="0 0 0" />
-      <mass
-        value="2" />
-      <inertia
-        ixx="0.480368573327889"
-        ixy="-2.89517779042653E-17"
-        ixz="-1.06691186966856E-17"
-        iyy="0.326889903542419"
-        iyz="-0.0724208623875704"
-        izz="0.60971027515868" />
+        xyz="1.66533453693773E-16 -0.804111102029834 0.0275105834465963"
+        rpy="0 0 0" />
+      <mass
+        value="27.2755326758408" />
+      <inertia
+        ixx="4.31133111414126"
+        ixy="6.65415782568477E-16"
+        ixz="-2.22750825253046E-16"
+        iyy="0.66836978637258"
+        iyz="-0.100077621756449"
+        izz="4.58294264392293" />
     </inertial>
     <visual>
@@ -472,5 +473,5 @@
     <inertial>
       <origin
-        xyz="2.22044604925031E-16 -1.11022302462516E-16 -0.0254"
+        xyz="0 8.32667268468867E-17 -0.0254"
         rpy="0 0 0" />
       <mass
@@ -478,9 +479,9 @@
       <inertia
         ixx="0.00460132751039961"
-        ixy="-5.42101086242752E-20"
-        ixz="3.41875854169894E-19"
+        ixy="-2.71050543121376E-20"
+        ixz="4.27969795118175E-19"
         iyy="0.00460132751039961"
-        iyz="1.20750969492291E-20"
-        izz="0.00850174046700707" />
+        iyz="1.30847375225861E-20"
+        izz="0.00850174046700706" />
     </inertial>
     <visual>
@@ -512,6 +513,6 @@
     type="continuous">
     <origin
-      xyz="-0.2286 -0.57366 -0.1651"
-      rpy="1.5708 0.042706 1.5708" />
+      xyz="-0.2286 -1.24477638939552 -0.1651"
+      rpy="1.5707963267949 0.0427063277818672 1.5707963267949" />
     <parent
       link="Trailer" />
@@ -525,5 +526,5 @@
     <inertial>
       <origin
-        xyz="0 -1.11022302462516E-16 0.0254"
+        xyz="0 8.32667268468867E-17 0.0253999999999999"
         rpy="0 0 0" />
       <mass
@@ -565,5 +566,5 @@
     type="continuous">
     <origin
-      xyz="0.2286 -0.57366 -0.1651"
+      xyz="0.2286 -1.2448 -0.1651"
       rpy="1.5708 0 1.5708" />
     <parent
@@ -574,3 +575,109 @@
       xyz="0 0 1" />
   </joint>
+  <link
+    name="Trailer_Left_Back_Wheel">
+    <inertial>
+      <origin
+        xyz="0 8.32667268468867E-17 -0.0254"
+        rpy="0 0 0" />
+      <mass
+        value="1.62962959682595" />
+      <inertia
+        ixx="0.00460132751039961"
+        ixy="-6.7762635780344E-20"
+        ixz="4.27969795118175E-19"
+        iyy="0.00460132751039961"
+        iyz="1.30847375225861E-20"
+        izz="0.00850174046700706" />
+    </inertial>
+    <visual>
+      <origin
+        xyz="0 0 0"
+        rpy="0 0 0" />
+      <geometry>
+        <mesh
+          filename="package://car_and_trailer/meshes/Trailer_Left_Back_Wheel.STL" />
+      </geometry>
+      <material
+        name="">
+        <color
+          rgba="0.792156862745098 0.819607843137255 0.933333333333333 1" />
+      </material>
+    </visual>
+    <collision>
+      <origin
+        xyz="0 0 0"
+        rpy="0 0 0" />
+      <geometry>
+        <mesh
+          filename="package://car_and_trailer/meshes/Trailer_Left_Back_Wheel.STL" />
+      </geometry>
+    </collision>
+  </link>
+  <joint
+    name="Trailer_Left_Back_Wheel_joint"
+    type="continuous">
+    <origin
+      xyz="-0.2286 -1.2448 -0.1651"
+      rpy="1.5708 0.042706 1.5708" />
+    <parent
+      link="Trailer" />
+    <child
+      link="Trailer_Left_Back_Wheel" />
+    <axis
+      xyz="0 0 1" />
+  </joint>
+  <link
+    name="Trailer_Right_Back_Wheel">
+    <inertial>
+      <origin
+        xyz="-2.22044604925031E-16 5.55111512312578E-17 0.0254"
+        rpy="0 0 0" />
+      <mass
+        value="1.62962959682594" />
+      <inertia
+        ixx="0.0046013275103996"
+        ixy="-7.56314231044298E-39"
+        ixz="3.36924666781802E-19"
+        iyy="0.0046013275103996"
+        iyz="-8.30428564488929E-36"
+        izz="0.00850174046700706" />
+    </inertial>
+    <visual>
+      <origin
+        xyz="0 0 0"
+        rpy="0 0 0" />
+      <geometry>
+        <mesh
+          filename="package://car_and_trailer/meshes/Trailer_Right_Back_Wheel.STL" />
+      </geometry>
+      <material
+        name="">
+        <color
+          rgba="0.792156862745098 0.819607843137255 0.933333333333333 1" />
+      </material>
+    </visual>
+    <collision>
+      <origin
+        xyz="0 0 0"
+        rpy="0 0 0" />
+      <geometry>
+        <mesh
+          filename="package://car_and_trailer/meshes/Trailer_Right_Back_Wheel.STL" />
+      </geometry>
+    </collision>
+  </link>
+  <joint
+    name="Trailer_Right_Back_Wheel_joint"
+    type="continuous">
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
Commit message: changes

File: car_and_trailer/urdf/car_and_trailer.urdf.xacro (robot description, xacro)
@@ -575,5 +575,5 @@
       xyz="0 0 1" />
   </joint>
-  <link
+  <!-- <link
     name="Trailer_Left_Back_Wheel">
     <inertial>
@@ -627,5 +627,5 @@
     <axis
       xyz="0 0 1" />
-  </joint>
+  </joint> -->
   <link
     name="Trailer_Right_Back_Wheel">

Commit message: controllers changes

File: car_and_trailer/urdf/car_and_trailer.urdf.xacro (robot description, xacro)
@@ -416,4 +416,39 @@
       xyz="0 0 1" />
   </joint>
+  <gazebo reference="Lidar">
+  <sensor name="lidar" type="ray">
+    <pose>0.0 0.0 0.0 0 0 0</pose>
+    <always_on>true</always_on>
+    <visualize>true</visualize>
+    <update_rate>5</update_rate>
+    <ray>
+      <scan>
+        <horizontal>
+          <samples>360</samples>
+          <resolution>1.00000</resolution>
+          <min_angle>0.000000</min_angle>
+          <max_angle>6.280000</max_angle>
+        </horizontal>
+      </scan>
+      <range>
+        <min>0.120000</min>
+        <max>3.5</max>
+        <resolution>0.015000</resolution>
+      </range>
+      <noise>
+        <type>gaussian</type>
+        <mean>0.0</mean>
+        <stddev>0.01</stddev>
+      </noise>
+    </ray>
+    <plugin name="scan" filename="libgazebo_ros_ray_sensor.so">
+      <ros>
+        <remapping>~/out:=scan</remapping>
+      </ros>
+      <output_type>sensor_msgs/LaserScan</output_type>
+      <frame_name>Lidar</frame_name>
+    </plugin>
+  </sensor>
+  </gazebo>
   <link
     name="Trailer">
@@ -473,5 +508,5 @@
     <inertial>
       <origin
-        xyz="0 8.32667268468867E-17 -0.0254"
+        xyz="0 4.32667268468867E-17 -0.0254"
         rpy="0 0 0" />
       <mass
@@ -513,5 +548,5 @@
     type="continuous">
     <origin
-      xyz="-0.2286 -1.24477638939552 -0.1651"
+      xyz="-0.2286 -0.44477638939552 -0.1651"
       rpy="1.5707963267949 0.0427063277818672 1.5707963267949" />
     <parent
@@ -526,5 +561,5 @@
     <inertial>
       <origin
-        xyz="0 8.32667268468867E-17 0.0253999999999999"
+        xyz="0 4.32667268468867E-17 0.0253999999999999"
         rpy="0 0 0" />
       <mass
@@ -566,5 +601,5 @@
     type="continuous">
     <origin
-      xyz="0.2286 -1.2448 -0.1651"
+      xyz="0.2286 -0.4448 -0.1651"
       rpy="1.5708 0 1.5708" />
     <parent
@@ -575,5 +610,5 @@
       xyz="0 0 1" />
   </joint>
-  <!-- <link
+  <link
     name="Trailer_Left_Back_Wheel">
     <inertial>
@@ -627,5 +662,5 @@
     <axis
       xyz="0 0 1" />
-  </joint> -->
+  </joint>
   <link
     name="Trailer_Right_Back_Wheel">
@@ -681,3 +716,43 @@
       xyz="0 0 1" />
   </joint>
+  <ros2_control name="GazeboSystem" type="system">
+    <hardware>
+        <plugin>gazebo_ros2_control/GazeboSystem</plugin>
+    </hardware>
+    <!-- # Velocity Controllers -->
+    <joint name="Rigth_Back_Wheel_joint">
+        <command_interface name="velocity">
+            <param name="min">-1000.0</param>
+            <param name="max">1000.0</param>
+        </command_interface>
+        <state_interface name="velocity"/>
+    </joint>
+    <joint name="Left_Back_Wheel_joint">
+        <command_interface name="velocity">
+            <param name="min">-1000.0</param>
+            <param name="max">1000.0</param>
+        </command_interface>
+        <state_interface name="velocity"/>
+    </joint>
+    <!-- # Position Controller -->
+    <joint name="Left_Front_Wheel_joint">
+        <command_interface name="position">
+            <param name="min">-3.14</param>
+            <param name="max">3.14</param>
+        </command_interface>
+        <state_interface name="position"/>
+    </joint>
+    <joint name="Rigth_Front_Wheel_joint">
+        <command_interface name="position">
+            <param name="min">-3.14</param>
+            <param name="max">3.14</param>
+        </command_interface>
+        <state_interface name="position"/>
+    </joint>
+</ros2_control>
+<gazebo>
+    <plugin filename="libgazebo_ros2_control.so" name="gazebo_ros2_control">
+        <parameters>$(find car_and_trailer)/config/control.yaml</parameters>
+    </plugin>
+</gazebo>
 </robot>

Commit message: added teleop

File: car_and_trailer/urdf/car_and_trailer.urdf.xacro (robot description, xacro)
@@ -721,5 +721,5 @@
     </hardware>
     <!-- # Velocity Controllers -->
-    <joint name="Rigth_Back_Wheel_joint">
+    <joint name="Right_Back_Wheel_joint">
         <command_interface name="velocity">
             <param name="min">-1000.0</param>
@@ -743,11 +743,4 @@
         <state_interface name="position"/>
     </joint>
-    <joint name="Rigth_Front_Wheel_joint">
-        <command_interface name="position">
-            <param name="min">-3.14</param>
-            <param name="max">3.14</param>
-        </command_interface>
-        <state_interface name="position"/>
-    </joint>
 </ros2_control>
 <gazebo>

Commit message: updated teleop

File: car_and_trailer/urdf/car_and_trailer.urdf.xacro (robot description, xacro)
@@ -743,4 +743,11 @@
         <state_interface name="position"/>
     </joint>
+    <joint name="Rigth_Front_Wheel_joint">
+        <command_interface name="position">
+            <param name="min">-3.14</param>
+            <param name="max">3.14</param>
+        </command_interface>
+        <state_interface name="position"/>
+    </joint>
 </ros2_control>
 <gazebo>
